Commit message: fix the model bug and add two joints controller

File: urdf/kinect.urdf.xacro (robot description, xacro)
@@ -36,5 +36,5 @@
         <origin xyz="0 0 0" rpy="0 0 1.5708"/>
         <geometry>
-          <mesh filename="package://simpledog/meshes/quadruped/kinect.dae" />
+          <mesh filename="package://simpledog/meshes/kinect.dae" />
         </geometry>
       </visual>

File: urdf/new_quadruped_model_kp.urdf.xacro (robot description, xacro)
@@ -50,10 +50,10 @@
         value="27.801" />
       <inertia
-        ixx="0.263947"
-        ixy="-0.003647"
-        ixz="0.009059"
-        iyy="2.018039"
-        iyz="-0.000762"
-        izz="2.056397" />
+        ixx="0.263893"
+        ixy="0"
+        ixz="0"
+        iyy="2.018032"
+        iyz="0"
+        izz="2.056458" />
     </inertial>
     <visual>
@@ -90,10 +90,10 @@
         value="2.9231" />
       <inertia
-        ixx="0.007845"
-        ixy="-0.00025"
-        ixz="-7.8E-05"
-        iyy="0.005144"
-        iyz="0.000967"
-        izz="0.00794" />
+        ixx="0.004820"
+        ixy="0"
+        ixz="0"
+        iyy="0.007868"
+        iyz="0"
+        izz="0.008241" />
     </inertial>
     <visual>
@@ -138,5 +138,4 @@
       lower="-3.0"
       upper="3.0"/>
-    <dynamics damping="0.7"/>
   </joint>
   <link
@@ -149,10 +148,10 @@
         value="4.2164" />
       <inertia
-        ixx="0.00627"
-        ixy="-0.000181"
-        ixz="-8.8E-05"
-        iyy="0.029233"
-        iyz="9.2E-05"
-        izz="0.028163" />
+        ixx="0.006286"
+        ixy="0"
+        ixz="0"
+        iyy="0.028156"
+        iyz="0"
+        izz="0.029242" />
     </inertial>
     <visual>
@@ -197,5 +196,4 @@
       lower="-7.0"
       upper="7.0"/>
-    <dynamics damping="0.7"/>
   </joint>
   <link
@@ -208,10 +206,10 @@
         value="0.44457" />
       <inertia
-        ixx="0.000397"
-        ixy="-4E-06"
-        ixz="0.000261"
-        iyy="0.0065"
-        iyz="-2.4E-05"
-        izz="0.006214" />
+        ixx="0.000385"
+        ixy="0"
+        ixz="0"
+        iyy="0.006223"
+        iyz="0"
+        izz="0.006502" />
     </inertial>
     <visual>
@@ -256,5 +254,4 @@
       lower="-3.0"
       upper="3.0"/>
-      <dynamics damping="0.7"/>
   </joint>
   <link
@@ -267,10 +264,10 @@
         value="0.03332" />
       <inertia
-        ixx="1.9126E-05"
-        ixy="-1.1072E-18"
-        ixz="-4.1175E-20"
-        iyy="0"
-        iyz="1.5428E-10"
-        izz="1.3678E-05" />
+        ixx="0.000014"
+        ixy="0"
+        ixz="0"
+        iyy="0.000014"
+        iyz="0"
+        izz="0.000019" />
     </inertial>
     <visual>
@@ -320,10 +317,10 @@
         value="2.923111" />
       <inertia
-        ixx="0.007845"
-        ixy="0.00025"
-        ixz="-7.8E-05"
-        iyy="0.005144"
-        iyz="-0.000967"
-        izz="0.00794" />
+        ixx="0.004820"
+        ixy="0"
+        ixz="0"
+        iyy="0.007868"
+        iyz="0"
+        izz="0.008241" />
     </inertial>
     <visual>
@@ -368,5 +365,4 @@
       lower="-3.0"
       upper="3.0"/>
-    <dynamics damping="0.7"/>
   </joint>
   <link
@@ -379,10 +375,10 @@
         value="4.216358" />
       <inertia
-        ixx="0.00627"
-        ixy="-0.000181"
-        ixz="-8.8E-05"
-        iyy="0.029233"
-        iyz="9.2E-05"
-        izz="0.028163" />
+        ixx="0.006286"
+        ixy="0"
+        ixz="0"
+        iyy="0.028156"
+        iyz="0"
+        izz="0.029242" />
     </inertial>
     <visual>
@@ -427,5 +423,4 @@
       lower="-7.0"
       upper="7.0"/>
-    <dynamics damping="0.7"/>
   </joint>
   <link
@@ -438,10 +433,10 @@
         value="0.444569" />
       <inertia
-        ixx="0.000397"
-        ixy="-4E-06"
-        ixz="0.000261"
-        iyy="0.0065"
-        iyz="-2.4E-05"
-        izz="0.006214" />
+        ixx="0.000385"
+        ixy="0"
+        ixz="0"
+        iyy="0.006223"
+        iyz="0"
+        izz="0.006502" />
     </inertial>
     <visual>
@@ -486,5 +481,4 @@
       lower="-3.0"
       upper="3.0"/>
-    <dynamics damping="0.7"/>
   </joint>
   <link
@@ -497,10 +491,10 @@
         value="0.03332" />
       <inertia
-        ixx="1.9126E-05"
-        ixy="-1.0162E-18"
-        ixz="-1.1377E-19"
-        iyy="1.3677E-05"
-        iyz="-6.5798E-11"
-        izz="1.3678E-05" />
+        ixx="0.000014"
+        ixy="0"
+        ixz="0"
+        iyy="0.000014"
+        iyz="0"
+        izz="0.000019" />
     </inertial>
     <visual>
@@ -529,5 +523,5 @@
   </link>
   <joint
-    name="rf_foot_Link"
+    name="rf_foot_joint"
     type="fixed">
     <origin
@@ -550,10 +544,10 @@
         value="2.9231" />
       <inertia
-        ixx="0.007845"
-        ixy="0.0025"
-        ixz="-7.8E-05"
-        iyy="0.005144"
-        iyz="-0.000967"
-        izz="0.00794" />
+        ixx="0.004820"
+        ixy="0"
+        ixz="0"
+        iyy="0.007868"
+        iyz="0"
+        izz="0.008241" />
     </inertial>
     <visual>
@@ -598,5 +592,4 @@
       lower="-3.0"
       upper="3.0"/>
-    <dynamics damping="0.7"/>
   </joint>
   <link
@@ -609,10 +602,10 @@
         value="4.216358" />
       <inertia
-        ixx="0.00627"
-        ixy="-0.000181"
-        ixz="-8.8E-05"
-        iyy="0.029233"
-        iyz="9.2E-05"
-        izz="0.028163" />
+        ixx="0.006286"
+        ixy="0"
+        ixz="0"
+        iyy="0.028156"
+        iyz="0"
+        izz="0.029242" />
     </inertial>
     <visual>
@@ -657,5 +650,4 @@
       lower="-7.0"
       upper="7.0"/>
-    <dynamics damping="0.7"/>
   </joint>
   <link
@@ -668,10 +660,10 @@
         value="0.444569" />
       <inertia
-        ixx="0.000397"
-        ixy="-4E-06"
-        ixz="-0.000261"
-        iyy="0.0065"
-        iyz="-2.4E-05"
-        izz="0.006214" />
+        ixx="0.000385"
+        ixy="0"
+        ixz="0"
+        iyy="0.006223"
+        iyz="0"
+        izz="0.006502" />
     </inertial>
     <visual>
@@ -716,5 +708,4 @@
       lower="-3.0"
       upper="3.0"/>
-    <dynamics damping="0.7"/>
   </joint>
   <link
@@ -727,10 +718,10 @@
         value="0.03332" />
       <inertia
-        ixx="1.9126E-05"
-        ixy="-9.3607E-19"
-        ixz="2.2915E-19"
-        iyy="1.3677E-05"
-        iyz="-2.7943E-10"
-        izz="1.3678E-05" />
+        ixx="0.000014"
+        ixy="0"
+        ixz="0"
+        iyy="0.000014"
+        iyz="0"
+        izz="0.000019" />
     </inertial>
     <visual>
@@ -780,10 +771,10 @@
         value="2.923111" />
       <inertia
-        ixx="0.007845"
-        ixy="-0.00025"
-        ixz="7.8E-05"
-        iyy="0.005144"
-        iyz="0.000967"
-        izz="0.00794" />
+        ixx="0.004820"
+        ixy="0"
+        ixz="0"
+        iyy="0.007868"
+        iyz="0"
+        izz="0.008241" />
     </inertial>
     <visual>
@@ -828,5 +819,4 @@
       lower="-3.0"
       upper="3.0"/>
-    <dynamics damping="0.7"/>
   </joint>
   <link
@@ -839,10 +829,10 @@
         value="4.216358" />
       <inertia
-        ixx="0.00627"
-        ixy="-0.000181"
-        ixz="-8.8E-05"
-        iyy="0.029233"
-        iyz="9.2E-05"
-        izz="0.028163" />
+        ixx="0.006286"
+        ixy="0"
+        ixz="0"
+        iyy="0.028156"
+        iyz="0"
+        izz="0.029242" />
     </inertial>
     <visual>
@@ -887,5 +877,4 @@
       lower="-7.0"
       upper="7.0"/>
-    <dynamics damping="0.7"/>
   </joint>
   <link
@@ -898,10 +887,10 @@
         value="0.444569" />
       <inertia
-        ixx="0.000397"
-        ixy="-4E-06"
-        ixz="0.000261"
-        iyy="0.0065"
-        iyz="-2.4E-05"
-        izz="0.006214" />
+        ixx="0.000385"
+        ixy="0"
+        ixz="0"
+        iyy="0.006223"
+        iyz="0"
+        izz="0.006502"/>
     </inertial>
     <visual>
@@ -946,5 +935,4 @@
       lower="-3.0"
       upper="3.0"/>
-    <dynamics damping="0.7"/>
   </joint>
   <link
@@ -957,10 +945,10 @@
         value="0.03332" />
       <inertia
-        ixx="1.9126E-05"
-        ixy="-9.5089E-19"
-        ixz="6.7668E-20"
-        iyy="1.3677E-05"
-        iyz="-2.7242E-10"
-        izz="1.3678E-05" />
+        ixx="0.000014"
+        ixy="0"
+        ixz="0"
+        iyy="0.000014"
+        iyz="0"
+        izz="0.000019" />
     </inertial>
     <visual>
@@ -1001,3 +989,3 @@
       xyz="0 0 0" />
   </joint>
-</robot>
+  </robot>
